File: mfo.kicad_pcb (KiCad board)
At the start: 2 copper layers, 19 x 15.2 mm, 21 parts, among them J1 S0, J2 Conn_01x04_Pin, J3 3V3_IN, J4 GND, J5 CLK1, J6 CLK2, J7 5V_IN, U1 TPS78218DDC, U2 CDCE925PWR, U3 TLV75733PDBV, Y1 27MHz

Commit message: add gerbers
Other:
- rule pad_to_mask_clearance: 0.05 -> 0
Changed lines of the file:
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@@
 			(dielectric_constraints no)
 		)
-		(pad_to_mask_clearance 0.05)
+		(pad_to_mask_clearance 0)
 		(allow_soldermask_bridges_in_footprints no)
 		(tenting front back)
 		(pcbplotparams
-			(layerselection 0x00000000_00000000_00000000_000000a5)
+			(layerselection 0x00000000_00000000_55555555_555575ff)
 			(plot_on_all_layers_selection 0x00000000_00000000_00000000_00000000)
 			(disableapertmacros no)
@@
 			(outputformat 1)
 			(mirror no)
-			(drillshape 1)
+			(drillshape 0)
 			(scaleselection 1)
-			(outputdirectory "")
+			(outputdirectory "gerbers/")
 		)
 	)

Commit message: fix
Other:
- board text added: "MULTIPLE FREQUENCY OSCILLATOR 3.3V/5V Original- skum Edit- yaruni github.com/owen-rp2a03/mfo"
- board text added: "Use only 1 source voltage, ensure correct one!"
- board text removed: "3.3V"
- board text removed: "MULTIPLE FREQUENCY OSCILLATOR 3V3/5V Original- skum Edit- yaruni"
Changed lines of the file:
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@@
 		(tenting front back)
 		(pcbplotparams
-			(layerselection 0x00000000_00000000_55555555_555575ff)
+			(layerselection 0x00000000_00000000_55555555_575575ff)
 			(plot_on_all_layers_selection 0x00000000_00000000_00000000_00000000)
 			(disableapertmacros no)
@@
 		)
 	)
-	(gr_text "MULTIPLE FREQUENCY\nOSCILLATOR 3V3/5V\nOriginal- skum\nEdit- yaruni"
-		(at 154.875 88.8 0)
+	(gr_text "MULTIPLE FREQUENCY\nOSCILLATOR 3.3V/5V\nOriginal- skum\nEdit- yaruni\ngithub.com/owen-rp2a03/mfo"
+		(at 154.559 91.948 0)
 		(layer "B.SilkS")
 		(effects
 			(font
-				(size 1 1)
-				(thickness 0.2)
+				(size 0.7 0.7)
+				(thickness 0.125)
+				(bold yes)
 			)
 			(justify left top mirror)
@@
 		)
 	)
-	(gr_text "3.3V"
-		(at 145.175 98.675 90)
+	(gr_text "3V3"
+		(at 145.034 98.933 90)
 		(layer "B.SilkS")
 		(effects
@@
 		)
 	)
+	(gr_text "Use only 1 source voltage, ensure correct one!"
+		(at 154.813 88.773 0)
+		(layer "B.SilkS")
+		(effects
+			(font
+				(size 0.7 0.5)
+				(thickness 0.125)
+			)
+			(justify left top mirror)
+		)
+	)
